Commit message: 20210531-1

File: demo_support/urdf/demo.xacro (robot description, xacro)
@@ -85,9 +85,4 @@
   </joint>
 -->
-  <!-- logical camera 1  model -->
-  <xacro:include filename="$(find demo_support)/urdf/logical_camera/logical_camera.urdf.xacro"/>
-  <xacro:logical_camera_urdf prefix="logical_camera1_" logical_camera_parent="world">
-    <origin xyz="0 0 1.0" rpy="0 1.5708 1.5708"/>
-  </xacro:logical_camera_urdf>
   <!-- robot1 to pedestal. -->
   <joint name="robot1_to_mountingplate_link" type="fixed">

Commit message: 20210601-2

File: demo_support/urdf/demo.xacro (robot description, xacro)
@@ -96,3 +96,9 @@
     <child link="vacuum_gripper1_base_link" />
   </joint>
+  <xacro:include filename="$(find pickit_model)/camera_description/urdf/pickit_camera_description.xacro"/>
+  <joint name="world_to camera" type="fixed">
+    <origin xyz="0 0 0.85" rpy="0 1.57 3.14"/>
+    <parent link="world" />
+    <child link="CAM_30703_link" />
+  </joint>
 </robot>
